File: enc_lego_pcb/enc_lego_v1_rev1.kicad_sch (KiCad schematic)
At the start: 8 parts, among them J1 BM05B-SRSS-TB_LF__SN_, J2 DNP, J3 Conn_01x02_Pin, U1 MT6701-SOP8

Commit message: updated BOM for order TS
Parts:
- C1: LCSC Part Number (none) -> C5120075
- D1: LCSC Part Number (none) -> C84260
- D2: LCSC Part Number (none) -> C908810
- J1: LCSC Part Number (none) -> C160391
- J3: value Conn_01x02_Pin -> DNP
- R1: LCSC Part Number (none) -> C3017846
- U1: LCSC Part Number (none) -> C2856764
Changed lines of the file:
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@@
       (effects (font (size 1.27 1.27)) hide)
     )
-    (property "Datasheet" "~" (at 136.525 67.31 0)
+    (property "Datasheet" "https://www.lcsc.com/product-detail/Chip-Resistor-Surface-Mount_VO-SCR0805J2K_C3017846.html" (at 136.525 67.31 0)
+      (effects (font (size 1.27 1.27)) hide)
+    )
+    (property "LCSC Part Number" "C3017846" (at 136.525 67.31 0)
       (effects (font (size 1.27 1.27)) hide)
     )
@@
       (effects (font (size 1.27 1.27)) (justify left bottom) hide)
     )
-    (property "Datasheet" "" (at 113.03 71.12 0)
+    (property "Datasheet" "https://www.lcsc.com/product-detail/Wire-To-Board-Connector_JST-BM05B-SRSS-TB-LF-SN_C160391.html" (at 113.03 71.12 0)
       (effects (font (size 1.27 1.27)) (justify left bottom) hide)
     )
@@
     (property "MANUFACTURER" "JST Sales America Inc." (at 113.03 71.12 0)
       (effects (font (size 1.27 1.27)) (justify left bottom) hide)
+    )
+    (property "LCSC Part Number" "C160391" (at 113.03 71.12 0)
+      (effects (font (size 1.27 1.27)) hide)
     )
     (pin "1")
@@
       (effects (font (size 1.27 1.27)) hide)
     )
-    (property "Datasheet" "" (at 63.5 72.39 0)
+    (property "Datasheet" "https://www.lcsc.com/product-detail/Position-Sensor_Magn-Tek-MT6701CT-STD_C2856764.html" (at 63.5 72.39 0)
+      (effects (font (size 1.27 1.27)) hide)
+    )
+    (property "LCSC Part Number" "C2856764" (at 63.5 72.39 0)
       (effects (font (size 1.27 1.27)) hide)
     )
@@
       (effects (font (size 1.27 1.27)) hide)
     )
+    (property "LCSC Part Number" "" (at 90.805 99.695 0)
+      (effects (font (size 1.27 1.27)) hide)
+    )
     (pin "1")
     (pin "2")
@@
       (effects (font (size 1.27 1.27)) (justify left bottom) hide)
     )
-    (property "Datasheet" "https://www.microsemi.com/document-portal/doc_download/135522-smaj-tvs-family-datasheet" (at -48.235 96.52 0)
+    (property "Datasheet" "https://www.lcsc.com/product-detail/Electrostatic-and-Surge-Protection-TVS-ESD_GOODWORK-SMAJ6-0CA_C908810.html" (at -48.235 96.52 0)
       (effects (font (size 1.27 1.27)) (justify left bottom) hide)
     )
@@
       (effects (font (size 1.27 1.27)) (justify left bottom) hide)
     )
+    (property "LCSC Part Number" "C908810" (at 145.415 83.82 0)
+      (effects (font (size 1.27 1.27)) hide)
+    )
     (pin "1")
     (pin "2")
@@
       (effects (font (size 1.27 1.27)) hide)
     )
-    (property "Datasheet" "~" (at 136.525 58.42 0)
+    (property "Datasheet" "https://www.lcsc.com/product-detail/Light-Emitting-Diodes-LED_Foshan-NationStar-Optoelectronics-NCD0805G1_C84260.html" (at 136.525 58.42 0)
+      (effects (font (size 1.27 1.27)) hide)
+    )
+    (property "LCSC Part Number" "C84260" (at 136.525 58.42 0)
       (effects (font (size 1.27 1.27)) hide)
     )
@@
       (effects (font (size 1.27 1.27)) (justify right))
     )
-    (property "Value" "Conn_01x02_Pin" (at 83.82 55.8799 0)
+    (property "Value" "DNP" (at 83.82 55.8799 0)
       (effects (font (size 1.27 1.27)) (justify right))
     )
@@
       (effects (font (size 1.27 1.27)) hide)
     )
+    (property "LCSC Part Number" "" (at 82.55 55.88 0)
+      (effects (font (size 1.27 1.27)) hide)
+    )
     (pin "1")
     (pin "2")
@@
       (effects (font (size 1.27 1.27)) hide)
     )
-    (property "Datasheet" "~" (at 135.255 93.98 0)
-      (effects (font (size 1.27 1.27)) hide)
-    )
+    (property "Datasheet" "https://www.lcsc.com/product-detail/Multilayer-Ceramic-Capacitors-MLCC-SMD-SMT_FH-Guangdong-Fenghua-Advanced-Tech-0805B104K250NT_C5120075.html" (at 135.255 93.98 0)
+      (effects (font (size 1.27 1.27)) hide)
+    )
+    (property "LCSC Part Number" "C5120075" (at 135.255 93.98 0)
+      (effects (font (size 1.27 1.27)) hide)
+    )
